File: Hardware/ESP32_minimal_WLED_sound.kicad_pcb (KiCad board)
At the start: 2 copper layers, 37.4 x 39.8 mm, 51 parts, among them J1 Conn_01x04_Male, J2 USB_C_Receptacle_USB2.0, J3 Conn_01x02_Male, J4 Barrel_Jack_Switch_Pin3Ring, J5 Conn_01x03_Male, J6 Conn_01x03_Male, J7 Conn_01x03_Male, J8 Conn_01x02_Male, J9 Conn_01x03_Male, Q1 AO3400A, SW2 Boot, U1 LMZM23601V5, U2 INA226, U3 LM1117-3.3, U4 TXS0102DCT, U5 ESP32-WROOM-32

Commit message: update button
Parts:
- removed SW2: Boot, Button_Switch_SMD:SW_SPST_B3U-1000P-B
- added SW1: SW_Push, Button_Switch_SMD:SW_Push_SPST_NO_Alps_SKRK, F.Cu at (128.3, 83.9)
- moved C6 0.08 mm to (131.8, 83.8)
Changed lines of the file:
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@@
     (48 "B.Fab" user)
     (49 "F.Fab" user)
-    (50 "User.1" user)
-    (51 "User.2" user)
-    (52 "User.3" user)
-    (53 "User.4" user)
-    (54 "User.5" user)
-    (55 "User.6" user)
-    (56 "User.7" user)
-    (57 "User.8" user)
-    (58 "User.9" user)
+    (50 "User.1" user "Nutzer.1")
+    (51 "User.2" user "Nutzer.2")
+    (52 "User.3" user "Nutzer.3")
+    (53 "User.4" user "Nutzer.4")
+    (54 "User.5" user "Nutzer.5")
+    (55 "User.6" user "Nutzer.6")
+    (56 "User.7" user "Nutzer.7")
+    (57 "User.8" user "Nutzer.8")
+    (58 "User.9" user "Nutzer.9")
   )
   (setup
@@
       (net 21 "SD") (pinfunction "SD") (pintype "output"))
   )
+  (footprint "Button_Switch_SMD:SW_Push_SPST_NO_Alps_SKRK" (layer "F.Cu")
+    (at 128.3 83.9 180)
+    (descr "http://www.alps.com/prod/info/E/HTML/Tact/SurfaceMount/SKRK/SKRKAHE020.html")
+    (tags "SMD SMT button")
+    (property "Sheetfile" "ESP32_minimal_WLED_sound.kicad_sch")
+    (property "Sheetname" "")
+    (attr smd)
+    (fp_text reference "SW1" (at 0 -2.25) (layer "F.SilkS")
+      (effects (font (size 0.7 0.7) (thickness 0.1)))
+    )
+    (fp_text value "SW_Push" (at 0 2.5) (layer "F.Fab")
+      (effects (font (size 1 1) (thickness 0.15)))
+    )
+    (fp_text user "${REFERENCE}" (at 0 0) (layer "F.Fab")
+      (effects (font (size 1 1) (thickness 0.15)))
+    )
+    (fp_line (start -2.07 1.57) (end -2.07 1.27) (layer "F.SilkS") (width 0.12))
+    (fp_line (start 2.07 1.27) (end 2.07 1.57) (layer "F.SilkS") (width 0.12))
+    (fp_line (start -2.07 -1.27) (end -2.07 -1.57) (layer "F.SilkS") (width 0.12))
+    (fp_line (start 2.07 -1.57) (end 2.07 -1.27) (layer "F.SilkS") (width 0.12))
+    (fp_line (start -2.07 -1.57) (end 2.07 -1.57) (layer "F.SilkS") (width 0.12))
+    (fp_line (start 2.07 1.57) (end -2.07 1.57) (layer "F.SilkS") (width 0.12))
+    (fp_line (start 2.75 1.7) (end -2.75 1.7) (layer "F.CrtYd") (width 0.05))
+    (fp_line (start -2.75 -1.7) (end 2.75 -1.7) (layer "F.CrtYd") (width 0.05))
+    (fp_line (start 2.75 -1.7) (end 2.75 1.7) (layer "F.CrtYd") (width 0.05))
+    (fp_line (start -2.75 1.7) (end -2.75 -1.7) (layer "F.CrtYd") (width 0.05))
+    (fp_line (start -1.95 -1.45) (end 1.95 -1.45) (layer "F.Fab") (width 0.1))
+    (fp_line (start 1.95 1.45) (end -1.95 1.45) (layer "F.Fab") (width 0.1))
+    (fp_line (start -1.95 1.45) (end -1.95 -1.45) (layer "F.Fab") (width 0.1))
+    (fp_line (start 1.95 -1.45) (end 1.95 1.45) (layer "F.Fab") (width 0.1))
+    (fp_circle (center 0 0) (end 1 0) (layer "F.Fab") (width 0.1) (fill none))
+    (pad "1" smd roundrect (at -2.1 0 180) (size 0.8 2) (layers "F.Cu" "F.Paste" "F.Mask") (roundrect_rratio 0.25)
+      (net 3 "IO00") (pinfunction "1") (pintype "passive"))
+    (pad "2" smd roundrect (at 2.1 0 180) (size 0.8 2) (layers "F.Cu" "F.Paste" "F.Mask") (roundrect_rratio 0.25)
+      (net 50 "GND") (pinfunction "2") (pintype "passive"))
+    (model "${KICAD6_3DMODEL_DIR}/Button_Switch_SMD.3dshapes/SW_Push_SPST_NO_Alps_SKRK.wrl"
+      (offset (xyz 0 0 0))
+      (scale (xyz 1 1 1))
+      (rotate (xyz 0 0 0))
+    )
+  )
   (footprint "TerminalBlock_Phoenix:TerminalBlock_Phoenix_MKDS-1,5-2-5.08_1x02_P5.08mm_Horizontal" (layer "F.Cu")
     (at 143.705 80.345 90)
@@
   )
   (footprint "Capacitor_SMD:C_0603_1608Metric" (layer "F.Cu")
-    (at 131.715095 83.840714 -90)
+    (at 131.8 83.840714 -90)
     (descr "Capacitor SMD 0603 (1608 Metric), square (rectangular) end terminal, IPC_7351 nominal, (Body size source: IPC-SM-782 page 76, https://www.pcb-3d.com/wordpress/wp-content/uploads/ipc-sm-782a_amendment_1_and_2.pdf), generated with kicad-footprint-generator")
     (tags "capacitor")
@@
       (offset (xyz 0 0 0))
       (scale (xyz 1 1 1))
-      (rotate (xyz 0 0 0))
-    )
-  )
-  (footprint "Button_Switch_SMD:SW_SPST_B3U-1000P-B" (layer "F.Cu")
-    (at 128.445285 83.79769)
-    (descr "Ultra-small-sized Tactile Switch with High Contact Reliability, Top-actuated Model, without Ground Terminal, with Boss")
-    (tags "Tactile Switch")
-    (property "LCSC" "C115357")
-    (property "Sheetfile" "ESP32_minimal_WLED_sound.kicad_sch")
-    (property "Sheetname" "")
-    (attr smd)
-    (fp_text reference "SW2" (at 0.054715 0.10231 180) (layer "F.SilkS")
-      (effects (font (size 0.7 0.7) (thickness 0.1)))
-    )
-    (fp_text value "Boot" (at 0.154715 2.00231 180) (layer "F.SilkS")
-      (effects (font (size 0.7 0.7) (thickness 0.1)))
-    )
-    (fp_text user "${REFERENCE}" (at 0 -2.5) (layer "F.Fab")
-      (effects (font (size 1 1) (thickness 0.15)))
-    )
-    (fp_line (start 1.65 1.4) (end 1.65 1.1) (layer "F.SilkS") (width 0.12))
-    (fp_line (start -1.65 1.1) (end -1.65 1.4) (layer "F.SilkS") (width 0.12))
-    (fp_line (start -1.65 -1.1) (end -1.65 -1.4) (layer "F.SilkS") (width 0.12))
-    (fp_line (start 1.65 -1.4) (end 1.65 -1.1) (layer "F.SilkS") (width 0.12))
-    (fp_line (start -1.65 -1.4) (end 1.65 -1.4) (layer "F.SilkS") (width 0.12))
-    (fp_line (start -1.65 1.4) (end 1.65 1.4) (layer "F.SilkS") (width 0.12))
-    (fp_line (start -2.4 1.65) (end 2.4 1.65) (layer "F.CrtYd") (width 0.05))
-    (fp_line (start 2.4 1.65) (end 2.4 -1.65) (layer "F.CrtYd") (width 0.05))
-    (fp_line (start 2.4 -1.65) (end -2.4 -1.65) (layer "F.CrtYd") (width 0.05))
-    (fp_line (start -2.4 -1.65) (end -2.4 1.65) (layer "F.CrtYd") (width 0.05))
-    (fp_line (start -1.5 -1.25) (end 1.5 -1.25) (layer "F.Fab") (width 0.1))
-    (fp_line (start -1.5 1.25) (end -1.5 -1.25) (layer "F.Fab") (width 0.1))
-    (fp_line (start 1.5 1.25) (end -1.5 1.25) (layer "F.Fab") (width 0.1))
-    (fp_line (start 1.5 -1.25) (end 1.5 1.25) (layer "F.Fab") (width 0.1))
-    (fp_circle (center 0 0) (end 0.75 0) (layer "F.Fab") (width 0.1) (fill none))
-    (pad "" np_thru_hole circle (at 0 0) (size 0.8 0.8) (drill 0.8) (layers *.Cu *.Mask))
-    (pad "1" smd rect (at -1.7 0) (size 0.9 1.7) (layers "F.Cu" "F.Paste" "F.Mask")
-      (net 50 "GND") (pinfunction "1") (pintype "passive"))
-    (pad "2" smd rect (at 1.7 0) (size 0.9 1.7) (layers "F.Cu" "F.Paste" "F.Mask")
-      (net 3 "IO00") (pinfunction "2") (pintype "passive"))
-    (model "${KICAD6_3DMODEL_DIR}/Button_Switch_SMD.3dshapes/SW_SPST_B3U-1000P-B.wrl"
-      (offset (xyz 0 0 0))
-      (scale (xyz 1 1 1))
